Commit message: Update eduexo.xacro

File: wearable_robot_description/urdf/eduexo.xacro (robot description, xacro)
@@ -13,6 +13,5 @@
         <visual>
             <geometry>
-                <!-- <mesh filename="package://wearable_robot_description/meshes/eduexo_base_link.dae" scale="0.01 0.01 0.01"/> -->
-                <mesh filename="/home/donghee/ros2_ws/src/wearable_robot_eval/wearable_robot_description/meshes/eduexo_base_link.dae" scale="0.01 0.01 0.01"/>
+                <mesh filename="$(find wearable_robot_description)/meshes/eduexo_base_link.dae" scale="0.01 0.01 0.01"/>
             </geometry>
             <origin rpy="0 0 0" xyz="0 0 0.6"/>
@@ -43,6 +42,5 @@
         <visual>
             <geometry>
-                <!-- <mesh filename="package://wearable_robot_description/meshes/eduexo_arm_link.dae" scale="0.01 0.01 0.01"/> -->
-                <mesh filename="/home/donghee/ros2_ws/src/wearable_robot_eval/wearable_robot_description/meshes/eduexo_arm_link.dae" scale="0.01 0.01 0.01"/>
+                <mesh filename="$(find wearable_robot_description)/meshes/eduexo_arm_link.dae" scale="0.01 0.01 0.01"/>
             </geometry>
             <origin rpy="0 -1.570796 0" xyz="0.0 0 0"/>
