Commit message: Make seperate 1 dof arm from human urdf

File: wearable_robot_description/urdf/1_dof_arm.xacro (robot description, xacro)
@@ -13,7 +13,7 @@
         <visual>
             <geometry>
-                <cylinder length="0.4" radius="0.04"/>
+                <cylinder length="0.3" radius="0.01"/>
             </geometry>
-            <origin rpy="0 0 0" xyz="0 0 0.6"/>
+            <origin rpy="0 0 1.570796" xyz="0.72 1 1.275"/>
             <material name="blue">
                 <color rgba="0 0 1 1"/>
@@ -22,7 +22,7 @@
         <collision>
             <geometry>
-                <cylinder length="0.4" radius="0.06"/>
+                <cylinder length="0.3" radius="0.01"/>
             </geometry>
-            <origin rpy="0 0 0" xyz="0 0 0.6"/>
+            <origin rpy="0 0 1.570796" xyz="0.72 1 1.275"/>
         </collision>
         <inertial>
@@ -34,7 +34,8 @@
         <parent link="base_link"/>
         <child link="arm_link"/>
-        <origin xyz="0 0 0.4"/>
-        <axis xyz="0 1 0" />
-        <limit effort="300" velocity="0.1" lower="4.71" upper="1.8"/>
+        <origin xyz="0.72 1 1.125"/>
+        <axis xyz="0 0 0" />
+        <!-- <limit effort="300" velocity="0.1" lower="4.71" upper="1.8"/> -->
+        <limit effort="300" velocity="0.1" lower="-4.1" upper="-1.5"/>
         <dynamics damping="50" friction="1"/>
     </joint>
@@ -42,7 +43,7 @@
         <visual>
             <geometry>
-                <cylinder length="0.4" radius="0.04"/>
+                <cylinder length="0.25" radius="0.01"/>
             </geometry>
-            <origin rpy="0 1.570796 0" xyz="-0.16 0 0"/>
+            <origin rpy="1.570796 0 0" xyz="0 0.125 0"/>
             <material name="red">
                 <color rgba="1 0 0 1"/>
@@ -51,7 +52,7 @@
         <collision>
             <geometry>
-                <cylinder length="0.4" radius="0.06"/>
+                <cylinder length="0.25" radius="0.01"/>
             </geometry>
-            <origin rpy="0 1.570796 0" xyz="-0.16 0 0"/>
+            <origin rpy="1.570796 0 0" xyz="0 0.125 0"/>
         </collision>
         <inertial>
@@ -59,4 +60,78 @@
             <inertia ixx="1.0" ixy="0.0" ixz="0.0" iyy="1.0" iyz="0.0" izz="1.0"/>
         </inertial>
+    </link>
+    <joint name="hand_link_fix_to_arm_link" type="fixed">
+      <origin xyz="0.12 0.18 0.05" rpy="0 1.570796 0"/>
+      <parent link="arm_link"/>
+      <child link="hand_link"/>
+    </joint>
+    <link name="hand_link">
+      <visual>
+        <geometry>
+          <cylinder length="0.01" radius="0.005"/>
+        </geometry>
+        <origin rpy="0 0 0" xyz="0 0 0"/>
+        <material name="red">
+          <color rgba="1 0 0 1"/>
+        </material>
+      </visual>
+      <visual>
+        <geometry>
+          <cylinder length="0.01" radius="0.005"/>
+        </geometry>
+        <origin rpy="0 0 0" xyz="0.1 0 0"/>
+        <material name="red">
+          <color rgba="1 0 0 1"/>
+        </material>
+      </visual>
+      <collision>
+        <geometry>
+          <cylinder length="0.05" radius="0.02"/>
+        </geometry>
+        <origin rpy="0 0 0" xyz="0 0 0"/>
+        <contact_coefficients mu="2.0" kp="2.0" kd="2.0" />
+      </collision>
+      <inertial>
+        <mass value="0.1"/>
+        <inertia ixx="1e-2" iyy="1e-2" izz="1e-2" ixy="0" ixz="0" iyz="0"/>
+      </inertial>
+    </link>
+    <joint name="hand_link_fix_to_base_link" type="fixed">
+      <!-- <origin xyz="0.12 0.19 0.05" rpy="0 1.570796 0"/> -->
+      <origin xyz="0.85 0.95 1.25" rpy="0 0 1.570796"/>
+      <axis xyz="0 0 0" />
+      <parent link="base_link"/>
+      <child link="hand_1_link"/>
+    </joint>
+    <link name="hand_1_link">
+      <visual>
+        <geometry>
+          <cylinder length="0.01" radius="0.005"/>
+        </geometry>
+        <origin rpy="0 0 0" xyz="0.0 0 0"/>
+        <material name="red">
+          <color rgba="1 0 0 1"/>
+        </material>
+      </visual>
+      <visual>
+        <geometry>
+          <cylinder length="0.01" radius="0.005"/>
+        </geometry>
+        <origin rpy="0 0 0" xyz="0.1 0 0"/>
+        <material name="red">
+          <color rgba="1 0 0 1"/>
+        </material>
+      </visual>
+      <collision>
+        <geometry>
+          <cylinder length="0.05" radius="0.005"/>
+        </geometry>
+        <origin rpy="0 0 0" xyz="0 0 0"/>
+        <contact_coefficients mu="2.0" kp="2.0" kd="2.0" />
+      </collision>
+      <inertial>
+        <mass value="0.1"/>
+        <inertia ixx="1e-2" iyy="1e-2" izz="1e-2" ixy="0" ixz="0" iyz="0"/>
+      </inertial>
     </link>
   <ros2_control name="GazeboSystem" type="system">
@@ -71,5 +146,4 @@
       <state_interface name="position"/>
       <state_interface name="velocity"/>
-      <state_interface name="effort"/>
     </joint>
   </ros2_control>

File: wearable_robot_description/urdf/human_66dof.xacro (robot description, xacro)
@@ -2,6 +2,5 @@
 <robot name="human" xmlns:xacro="http://www.ros.org/wiki/xacro">
   <!-- Import all Gazebo-customization elements, including Gazebo colors -->
-  <xacro:include filename="$(find wearable_robot_description)/urdf/human.gazebo"/>
-  <xacro:include filename="$(find wearable_robot_description)/urdf/1_dof_arm.gazebo"/>
+  <!-- <xacro:include filename="$(find wearable_robot_description)/urdf/human_66dof.gazebo"/> -->
   <!-- Import Rviz colors -->
   <xacro:include filename="$(find wearable_robot_description)/urdf/materials.xacro"/>
@@ -11,14 +10,14 @@
     <!--   <child link="base_link"/> -->
     <!-- </joint> -->
-    <joint name="base_link_fix_to_right_upper_arm" type="fixed">
-      <origin xyz="0    -0.27          0.1" rpy="0 1.570796 1.570796"/>
-      <parent link="RightUpperArm"/>
-      <child link="base_link"/>
-    </joint>
-    <joint name="hand_link_fix_to_arm_link" type="fixed">
-      <origin xyz="0.05    +0.35          0.1" rpy="0 1.570796 0"/>
-      <parent link="arm_link"/>
-      <child link="hand_link"/>
-    </joint>
+    <!-- <joint name="base_link_fix_to_right_upper_arm" type="fixed"> -->
+    <!--   <origin xyz="0    -0.27          0.1" rpy="0 1.570796 1.570796"/> -->
+    <!--   <parent link="RightUpperArm"/> -->
+    <!--   <child link="base_link"/> -->
+    <!-- </joint> -->
+    <!-- <joint name="hand_link_fix_to_arm_link" type="fixed"> -->
+    <!--   <origin xyz="0.05    +0.35          0.1" rpy="0 1.570796 0"/> -->
+    <!--   <parent link="arm_link"/> -->
+    <!--   <child link="hand_link"/> -->
+    <!-- </joint> -->
     <!-- <joint name="RightHand_fixed" type="fixed"> -->
     <!--   <origin xyz="0 0 0" rpy="0 0 0"/> -->
@@ -31,117 +30,85 @@
     <!--   <child link="hand_link"/> -->
     <!-- </joint> -->
-    <link name="base_link">
-        <visual>
-            <geometry>
-                <cylinder length="0.4" radius="0.04"/>
-            </geometry>
-            <origin rpy="0 0 0" xyz="0 0 0.2"/>
-            <material name="blue">
-                <color rgba="0 0 1 1"/>
-            </material>
-        </visual>
-        <collision>
-            <geometry>
-                <cylinder length="0.4" radius="0.06"/>
-            </geometry>
-            <origin rpy="0 0 0" xyz="0 0 0.2"/>
-        </collision>
-        <inertial>
-            <mass value="0.1"/>
-            <inertia ixx="1e-2" iyy="1e-2" izz="1e-2" ixy="0" ixz="0" iyz="0"/>
-        </inertial>
-    </link>
-    <joint name="arm_joint" type="revolute">
-        <parent link="base_link"/>
-        <child link="arm_link"/>
-        <!-- <origin xyz="0 0 1.0"/> -->
-        <origin xyz="0 0 0"/>
-        <axis xyz="1 0 0" />
-        <limit effort="300" velocity="0.1" lower="4.71" upper="1.8"/>
-        <dynamics damping="50" friction="1"/>
-    </joint>
-    <link name="arm_link">
-        <visual>
-            <geometry>
-                <cylinder length="0.4" radius="0.04"/>
-            </geometry>
-            <!-- <origin rpy="0 1.570796 0" xyz="-0.16 0 0"/> -->
-            <!-- <origin rpy="0 1.570796 0" xyz="0 0 0"/> -->
-            <origin rpy="1.570796 0 0" xyz="0 0.2 0"/>
-            <material name="red">
-                <color rgba="1 0 0 1"/>
-            </material>
-        </visual>
-        <collision>
-            <geometry>
-                <cylinder length="0.4" radius="0.06"/>
-            </geometry>
-            <!-- <origin rpy="0 1.570796 0" xyz="-0.16 0 0"/> -->
-            <!-- <origin rpy="0 1.570796 0" xyz="0 0 0"/> -->
-            <origin rpy="1.570796 0 0" xyz="0 0.2 0"/>
-        </collision>
-        <inertial>
-            <mass value="0.1"/>
-            <inertia ixx="1e-2" iyy="1e-2" izz="1e-2" ixy="0" ixz="0" iyz="0"/>
-        </inertial>
-    </link>
-    <link name="hand_link">
-        <visual>
-            <geometry>
-                <cylinder length="0.15" radius="0.04"/>
-            </geometry>
-            <origin rpy="0 0 0" xyz="0 0 0"/>
-            <!-- <origin rpy="0 0 0" xyz="0 -0.2 0"/> -->
-            <material name="red">
-                <color rgba="1 0 0 1"/>
-            </material>
-        </visual>
-        <collision>
-            <geometry>
-                <cylinder length="0.15" radius="0.04"/>
-            </geometry>
-            <!-- <origin rpy="0 1.570796 0" xyz="-0.16 0 0"/> -->
-            <!-- <origin rpy="0 1.570796 0" xyz="0 0 0"/> -->
-            <origin rpy="0 0 0" xyz="0 0 0"/>
-            <!-- <contact_coefficients mu="2.0" kp="2.0" kd="2.0" /> -->
-            <contact_coefficients mu="0" kp="1000.0" kd="1.0"/>
-        </collision>
-        <inertial>
-            <mass value="0.1"/>
-            <inertia ixx="1e-2" iyy="1e-2" izz="1e-2" ixy="0" ixz="0" iyz="0"/>
-        </inertial>
-    </link>
-  <ros2_control name="GazeboSystem" type="system">
-    <hardware>
-      <plugin>gazebo_ros2_control/GazeboSystem</plugin>
-    </hardware>
-    <joint name="arm_joint">
-      <command_interface name="position">
-        <param name="min">1.79</param>
-        <param name="max">6.28</param>
-      </command_interface>
-      <!-- <command_interface name="velocity"> -->
-      <!--   <param name="min">-5</param> -->
-      <!--   <param name="max">5</param> -->
-      <!-- </command_interface> -->
-      <state_interface name="position"/>
-      <state_interface name="velocity"/>
-      <state_interface name="effort"/>
-    </joint>
-  </ros2_control>
-  <!-- <ros2_control name="GazeboSystem" type="system"> -->
-  <!--   <hardware> -->
-  <!--     <plugin>gazebo_ros2_control/GazeboSystem</plugin> -->
-  <!--   </hardware> -->
-  <!--   <joint name="jRightElbow_rotx"> -->
-  <!--     <command_interface name="position"> -->
-  <!--       <param name="min">1.79</param> -->
-  <!--       <param name="max">6.28</param> -->
-  <!--     </command_interface> -->
-  <!--     <state_interface name="position"/> -->
-  <!--     <state_interface name="velocity"/> -->
-  <!--     <state_interface name="acceleration"/> -->
+  <!--   <link name="base_link"> -->
+  <!--       <visual> -->
+  <!--           <geometry> -->
+  <!--               <cylinder length="0.4" radius="0.04"/> -->
+  <!--           </geometry> -->
+  <!--           <origin rpy="0 0 0" xyz="0 0 0.2"/> -->
+  <!--           <material name="blue"> -->
+  <!--               <color rgba="0 0 1 1"/> -->
+  <!--           </material> -->
+  <!--       </visual> -->
+  <!--       <collision> -->
+  <!--           <geometry> -->
+  <!--               <cylinder length="0.4" radius="0.06"/> -->
+  <!--           </geometry> -->
+  <!--           <origin rpy="0 0 0" xyz="0 0 0.2"/> -->
+  <!--       </collision> -->
+  <!--       <inertial> -->
+  <!--           <mass value="0.1"/> -->
+  <!--           <inertia ixx="1e-2" iyy="1e-2" izz="1e-2" ixy="0" ixz="0" iyz="0"/> -->
+  <!--       </inertial> -->
+  <!--   </link> -->
+  <!--   <joint name="arm_joint" type="revolute"> -->
+  <!--       <parent link="base_link"/> -->
+  <!--       <child link="arm_link"/> -->
+  <!--       <!-\- <origin xyz="0 0 1.0"/> -\-> -->
+  <!--       <origin xyz="0 0 0"/> -->
+  <!--       <axis xyz="1 0 0" /> -->
+  <!--       <limit effort="300" velocity="0.1" lower="4.71" upper="1.8"/> -->
+  <!--       <dynamics damping="50" friction="1"/> -->
   <!--   </joint> -->
-  <!-- </ros2_control> -->
+  <!--   <link name="arm_link"> -->
+  <!--       <visual> -->
+  <!--           <geometry> -->
+  <!--               <cylinder length="0.4" radius="0.04"/> -->
+  <!--           </geometry> -->
+  <!--           <!-\- <origin rpy="0 1.570796 0" xyz="-0.16 0 0"/> -\-> -->
+  <!--           <!-\- <origin rpy="0 1.570796 0" xyz="0 0 0"/> -\-> -->
+  <!--           <origin rpy="1.570796 0 0" xyz="0 0.2 0"/> -->
+  <!--           <material name="red"> -->
+  <!--               <color rgba="1 0 0 1"/> -->
+  <!--           </material> -->
+  <!--       </visual> -->
+  <!--       <collision> -->
+  <!--           <geometry> -->
+  <!--               <cylinder length="0.4" radius="0.06"/> -->
+  <!--           </geometry> -->
+  <!--           <!-\- <origin rpy="0 1.570796 0" xyz="-0.16 0 0"/> -\-> -->
+  <!--           <!-\- <origin rpy="0 1.570796 0" xyz="0 0 0"/> -\-> -->
+  <!--           <origin rpy="1.570796 0 0" xyz="0 0.2 0"/> -->
+  <!--       </collision> -->
+  <!--       <inertial> -->
+  <!--           <mass value="0.1"/> -->
+  <!--           <inertia ixx="1e-2" iyy="1e-2" izz="1e-2" ixy="0" ixz="0" iyz="0"/> -->
+  <!--       </inertial> -->
+  <!--   </link> -->
+  <!--   <link name="hand_link"> -->
+  <!--       <visual> -->
+  <!--           <geometry> -->
+  <!--               <cylinder length="0.15" radius="0.04"/> -->
+  <!--           </geometry> -->
+  <!--           <origin rpy="0 0 0" xyz="0 0 0"/> -->
+  <!--           <!-\- <origin rpy="0 0 0" xyz="0 -0.2 0"/> -\-> -->
+  <!--           <material name="red"> -->
+  <!--               <color rgba="1 0 0 1"/> -->
+  <!--           </material> -->
+  <!--       </visual> -->
+  <!--       <collision> -->
+  <!--           <geometry> -->
+  <!--               <cylinder length="0.15" radius="0.04"/> -->
+  <!--           </geometry> -->
+  <!--           <!-\- <origin rpy="0 1.570796 0" xyz="-0.16 0 0"/> -\-> -->
+  <!--           <!-\- <origin rpy="0 1.570796 0" xyz="0 0 0"/> -\-> -->
+  <!--           <origin rpy="0 0 0" xyz="0 0 0"/> -->
+  <!--           <!-\- <contact_coefficients mu="2.0" kp="2.0" kd="2.0" /> -\-> -->
+  <!--           <contact_coefficients mu="0" kp="1000.0" kd="1.0"/> -->
+  <!--       </collision> -->
+  <!--       <inertial> -->
+  <!--           <mass value="0.1"/> -->
+  <!--           <inertia ixx="1e-2" iyy="1e-2" izz="1e-2" ixy="0" ixz="0" iyz="0"/> -->
+  <!--       </inertial> -->
+  <!--   </link> -->
   <!--To open this model with Gazebo replace the null masses, inertias and dimensions of the 'fake links f1 and f2'-->
   <!--LINKS-->
@@ -1574,4 +1541,17 @@
     <origin xyz="1 1 0.95" rpy="0 0 ${-0.5*pi}" />
   </joint>
+  <ros2_control name="GazeboSystem" type="system">
+    <hardware>
+      <plugin>gazebo_ros2_control/GazeboSystem</plugin>
+    </hardware>
+    <joint name="jRightElbow_rotx">
+      <command_interface name="position">
+        <param name="min">1.79</param>
+        <param name="max">6.28</param>
+      </command_interface>
+      <state_interface name="position"/>
+      <state_interface name="velocity"/>
+    </joint>
+  </ros2_control>
   <!-- Sensor  1-->
   <sensor name="Pelvis_gyro" type="gyroscope">
@@ -1725,5 +1705,5 @@
   <sensor name="LeftFoot_accelerometer" type="accelerometer">
     <parent link="LeftFoot"/>
-    <origin xyz="0.083701  -0.0013929   -0.011817" rpy="-0.10862      0.4501     0.37976"/>
+p    <origin xyz="0.083701  -0.0013929   -0.011817" rpy="-0.10862      0.4501     0.37976"/>
   </sensor>
 </robot>

Commit message: Rename link names

File: wearable_robot_description/urdf/1_dof_arm.xacro (robot description, xacro)
@@ -8,7 +8,7 @@
     <joint name="fixed" type="fixed">
         <parent link="world"/>
-        <child link="base_link"/>
+        <child link="arm_link"/>
     </joint>
-    <link name="base_link">
+    <link name="arm_link">
         <visual>
             <geometry>
@@ -27,11 +27,11 @@
         </collision>
         <inertial>
-            <mass value="1"/>
+            <mass value="0.5"/>
             <inertia ixx="1.0" ixy="0.0" ixz="0.0" iyy="1.0" iyz="0.0" izz="1.0"/>
         </inertial>
     </link>
     <joint name="arm_joint" type="revolute">
-        <parent link="base_link"/>
-        <child link="arm_link"/>
+        <parent link="arm_link"/>
+        <child link="forearm_link"/>
         <origin xyz="0.72 1 1.125"/>
         <axis xyz="0 0 0" />
@@ -40,5 +40,5 @@
         <dynamics damping="50" friction="1"/>
     </joint>
-    <link name="arm_link">
+    <link name="forearm_link">
         <visual>
             <geometry>
@@ -57,14 +57,14 @@
         </collision>
         <inertial>
-            <mass value="1"/>
+            <mass value="0.5"/>
             <inertia ixx="1.0" ixy="0.0" ixz="0.0" iyy="1.0" iyz="0.0" izz="1.0"/>
         </inertial>
     </link>
-    <joint name="hand_link_fix_to_arm_link" type="fixed">
+    <joint name="forearm_band_link_fix_to_forearm_link" type="fixed">
       <origin xyz="0.12 0.18 0.05" rpy="0 1.570796 0"/>
-      <parent link="arm_link"/>
-      <child link="hand_link"/>
+      <parent link="forearm_link"/>
+      <child link="forearm_band_link"/>
     </joint>
-    <link name="hand_link">
+    <link name="forearm_band_link">
       <visual>
         <geometry>
@@ -92,4 +92,11 @@
         <contact_coefficients mu="2.0" kp="2.0" kd="2.0" />
       </collision>
+      <collision>
+        <geometry>
+          <cylinder length="0.05" radius="0.02"/>
+        </geometry>
+        <origin rpy="0 0 0" xyz="0.1 0 0"/>
+        <contact_coefficients mu="2.0" kp="2.0" kd="2.0" />
+      </collision>
       <inertial>
         <mass value="0.1"/>
@@ -97,12 +104,12 @@
       </inertial>
     </link>
-    <joint name="hand_link_fix_to_base_link" type="fixed">
+    <joint name="arm_band_link_fix_to_arm_link" type="fixed">
       <!-- <origin xyz="0.12 0.19 0.05" rpy="0 1.570796 0"/> -->
       <origin xyz="0.85 0.95 1.25" rpy="0 0 1.570796"/>
       <axis xyz="0 0 0" />
-      <parent link="base_link"/>
-      <child link="hand_1_link"/>
+      <parent link="arm_link"/>
+      <child link="arm_band_link"/>
     </joint>
-    <link name="hand_1_link">
+    <link name="arm_band_link">
       <visual>
         <geometry>
@@ -110,4 +117,13 @@
         </geometry>
         <origin rpy="0 0 0" xyz="0.0 0 0"/>
+        <material name="red">
+          <color rgba="1 0 0 1"/>
+        </material>
+      </visual>
+      <visual>
+        <geometry>
+          <cylinder length="0.01" radius="0.005"/>
+        </geometry>
+        <origin rpy="0 0 0" xyz="0.05 0 0.225"/>
         <material name="red">
           <color rgba="1 0 0 1"/>
@@ -128,4 +144,18 @@
         </geometry>
         <origin rpy="0 0 0" xyz="0 0 0"/>
+        <contact_coefficients mu="2.0" kp="2.0" kd="2.0" />
+      </collision>
+      <collision>
+        <geometry>
+          <cylinder length="0.05" radius="0.005"/>
+        </geometry>
+        <origin rpy="0 0 0" xyz="0.05 0 0.225"/>
+        <contact_coefficients mu="2.0" kp="2.0" kd="2.0" />
+      </collision>
+      <collision>
+        <geometry>
+          <cylinder length="0.05" radius="0.005"/>
+        </geometry>
+        <origin rpy="0 0 0" xyz="0.1 0 0"/>
         <contact_coefficients mu="2.0" kp="2.0" kd="2.0" />
       </collision>

Commit message: Update 1 dof arm urdf

File: wearable_robot_description/urdf/1_dof_arm.xacro (robot description, xacro)
@@ -125,13 +125,4 @@
           <cylinder length="0.01" radius="0.005"/>
         </geometry>
-        <origin rpy="0 0 0" xyz="0.05 0 0.225"/>
-        <material name="red">
-          <color rgba="1 0 0 1"/>
-        </material>
-      </visual>
-      <visual>
-        <geometry>
-          <cylinder length="0.01" radius="0.005"/>
-        </geometry>
         <origin rpy="0 0 0" xyz="0.1 0 0"/>
         <material name="red">
@@ -144,11 +135,4 @@
         </geometry>
         <origin rpy="0 0 0" xyz="0 0 0"/>
-        <contact_coefficients mu="2.0" kp="2.0" kd="2.0" />
-      </collision>
-      <collision>
-        <geometry>
-          <cylinder length="0.05" radius="0.005"/>
-        </geometry>
-        <origin rpy="0 0 0" xyz="0.05 0 0.225"/>
         <contact_coefficients mu="2.0" kp="2.0" kd="2.0" />
       </collision>

Commit message: Fix 1 dof arm urdf collision size

File: wearable_robot_description/urdf/1_dof_arm.xacro (robot description, xacro)
@@ -71,5 +71,5 @@
           <cylinder length="0.01" radius="0.005"/>
         </geometry>
-        <origin rpy="0 0 0" xyz="0 0 0"/>
+        <origin rpy="0 0 0" xyz="0.01 0 0"/>
         <material name="red">
           <color rgba="1 0 0 1"/>
@@ -80,5 +80,5 @@
           <cylinder length="0.01" radius="0.005"/>
         </geometry>
-        <origin rpy="0 0 0" xyz="0.1 0 0"/>
+        <origin rpy="0 0 0" xyz="0.09 0 0"/>
         <material name="red">
           <color rgba="1 0 0 1"/>
@@ -87,14 +87,14 @@
       <collision>
         <geometry>
-          <cylinder length="0.05" radius="0.02"/>
+          <cylinder length="0.02" radius="0.005"/>
         </geometry>
-        <origin rpy="0 0 0" xyz="0 0 0"/>
+        <origin rpy="0 0 0" xyz="0.01 0 0"/>
         <contact_coefficients mu="2.0" kp="2.0" kd="2.0" />
       </collision>
       <collision>
         <geometry>
-          <cylinder length="0.05" radius="0.02"/>
+          <cylinder length="0.02" radius="0.005"/>
         </geometry>
-        <origin rpy="0 0 0" xyz="0.1 0 0"/>
+        <origin rpy="0 0 0" xyz="0.09 0 0"/>
         <contact_coefficients mu="2.0" kp="2.0" kd="2.0" />
       </collision>
@@ -116,5 +116,5 @@
           <cylinder length="0.01" radius="0.005"/>
         </geometry>
-        <origin rpy="0 0 0" xyz="0.0 0 0"/>
+        <origin rpy="1.570796 0 0" xyz="0.01 0 0"/>
         <material name="red">
           <color rgba="1 0 0 1"/>
@@ -125,5 +125,5 @@
           <cylinder length="0.01" radius="0.005"/>
         </geometry>
-        <origin rpy="0 0 0" xyz="0.1 0 0"/>
+        <origin rpy="1.570796 0 0" xyz="0.09 0 0"/>
         <material name="red">
           <color rgba="1 0 0 1"/>
@@ -132,14 +132,14 @@
       <collision>
         <geometry>
-          <cylinder length="0.05" radius="0.005"/>
+          <cylinder length="0.02" radius="0.005"/>
         </geometry>
-        <origin rpy="0 0 0" xyz="0 0 0"/>
+        <origin rpy="1.570796 0 0" xyz="0.01 0 0"/>
         <contact_coefficients mu="2.0" kp="2.0" kd="2.0" />
       </collision>
       <collision>
         <geometry>
-          <cylinder length="0.05" radius="0.005"/>
+          <cylinder length="0.02" radius="0.005"/>
         </geometry>
-        <origin rpy="0 0 0" xyz="0.1 0 0"/>
+        <origin rpy="1.570796 0 0" xyz="0.09 0 0"/>
         <contact_coefficients mu="2.0" kp="2.0" kd="2.0" />
       </collision>
