Commit message: Make human_66dof model visible in gazebo

File: wearable_robot_description/urdf/human_66dof.xacro (robot description, xacro)
@@ -1,1580 +1,1587 @@
 <!--URDF MODEL 66 DoFs-->
-<robot name="XSensStyleModel_template">
-<material name="color">
-    <color rgba="0.1 0.1 0.1 1"/>
-</material>
-<!--To open this model with Gazebo replace the null masses, inertias and dimensions of the 'fake links f1 and f2'-->
-    <!--LINKS-->
-	<!--Link base (1)-->
-	<link name="Pelvis">
-        <inertial>
-            <mass value="4.976"/>
-			<!--COM origin wrt pHipOrigin-->
-            <origin xyz="0           0    0.049743" rpy="0 0 0" />
-            <inertia ixx="0.029678" iyy="0.011854" izz="0.033653" ixy="0" ixz="0" iyz="0"/>
-        </inertial>
-        <visual>
-			<!--box origin wrt pHipOrigin-->
-            <origin xyz="0           0    0.049743" rpy="0 0 0" />
-            <geometry>
-                <box size="0.13815     0.24914    0.097469"/>
-            </geometry>
-            <material name="color"/>
-        </visual>
-        <collision>
-			<!--box origin wrt pHipOrigin-->
-            <origin xyz="0           0    0.049743" rpy="0 0 0" />
-            <geometry>
-                <box size="0.13815     0.24914    0.097469"/>
-            </geometry>
-        </collision>
-    </link>
-    <!--Chain from (2) to (7)-->
-	<link name="L5_f1">
-        <inertial>
-            <mass value="0"/>
-            <origin xyz="0 0 0" rpy="0 0 0" />
-            <inertia ixx="0" iyy="0" izz="0" ixy="0" ixz="0" iyz="0"/>
-        </inertial>
-    </link>
-	<link name="L5_f2">
-        <inertial>
-            <mass value="0"/>
-            <origin xyz="0 0 0" rpy="0 0 0" />
-            <inertia ixx="0" iyy="0" izz="0" ixy="0" ixz="0" iyz="0"/>
-        </inertial>
-    </link>
-	<link name="L5">
-        <inertial>
-            <mass value="6.3444"/>
-			<!--COM origin wrt jL5S1-->
-            <origin xyz="0           0    0.047552" rpy="0 0 0" />
-            <inertia ixx="0.018868" iyy="0.014872" izz="0.024177" ixy="0" ixz="0" iyz="0"/>
-        </inertial>
-        <visual>
-			<!--box origin origin wrt jL5S1-->
-            <origin xyz="0           0    0.047552" rpy="0 0 0" />
-            <geometry>
-                <box size="0.13815     0.16323    0.095104"/>
-            </geometry>
-            <material name="color"/>
-        </visual>
-        <collision>
-			<!--box origin origin wrt jL5S1-->
-            <origin xyz="0           0    0.047552" rpy="0 0 0" />
-            <geometry>
-                <box size="0.13815     0.16323    0.095104"/>
-            </geometry>
-        </collision>
-    </link>
-	<link name="L3_f1">
-        <inertial>
-            <mass value="0"/>
-            <origin xyz="0 0 0" rpy="0 0 0" />
-            <inertia ixx="0" iyy="0" izz="0" ixy="0" ixz="0" iyz="0"/>
-        </inertial>
-    </link>
-	<link name="L3_f2">
-        <inertial>
-            <mass value="0"/>
-            <origin xyz="0 0 0" rpy="0 0 0" />
-            <inertia ixx="0" iyy="0" izz="0" ixy="0" ixz="0" iyz="0"/>
-        </inertial>
-    </link>
-	<link name="L3">
-        <inertial>
-            <mass value="6.3444"/>
-			<!--COM origin wrt jL4L3-->
-            <origin xyz="0           0    0.042958" rpy="0 0 0" />
-            <inertia ixx="0.017989" iyy="0.013993" izz="0.024177" ixy="0" ixz="0" iyz="0"/>
-        </inertial>
-        <visual>
-			<!--box origin origin wrt jL4L3-->
-            <origin xyz="0           0    0.042958" rpy="0 0 0" />
-            <geometry>
-                <box size="0.13815     0.16323    0.085916"/>
-            </geometry>
-            <material name="color"/>
-        </visual>
-        <collision>
-			<!--box origin origin wrt jL4L3-->
-            <origin xyz="0           0    0.042958" rpy="0 0 0" />
-            <geometry>
-                <box size="0.13815     0.16323    0.085916"/>
-            </geometry>
-        </collision>
-    </link>
-	<link name="T12_f1">
-        <inertial>
-            <mass value="0"/>
-            <origin xyz="0 0 0" rpy="0 0 0" />
-            <inertia ixx="0" iyy="0" izz="0" ixy="0" ixz="0" iyz="0"/>
-        </inertial>
-    </link>
-	<link name="T12_f2">
-        <inertial>
-            <mass value="0"/>
-            <origin xyz="0 0 0" rpy="0 0 0" />
-            <inertia ixx="0" iyy="0" izz="0" ixy="0" ixz="0" iyz="0"/>
-        </inertial>
-    </link>
-	<link name="T12">
-        <inertial>
-            <mass value="6.3444"/>
-			<!--COM origin wrt jL1T12-->
-            <origin xyz="0           0    0.042958" rpy="0 0 0" />
-            <inertia ixx="0.017989" iyy="0.013993" izz="0.024177" ixy="0" ixz="0" iyz="0"/>
-        </inertial>
-        <visual>
-			<!--box origin origin wrt jL1T12-->
-            <origin xyz="0           0    0.042958" rpy="0 0 0" />
-            <geometry>
-                <box size="0.13815     0.16323    0.085916"/>
-            </geometry>
-            <material name="color"/>
-        </visual>
-        <collision>
-			<!--box origin origin wrt jL1T12-->
-            <origin xyz="0           0    0.042958" rpy="0 0 0" />
-            <geometry>
-                <box size="0.13815     0.16323    0.085916"/>
-            </geometry>
-        </collision>
-    </link>
-	<link name="T8_f1">
-        <inertial>
-            <mass value="0"/>
-            <origin xyz="0 0 0" rpy="0 0 0" />
-            <inertia ixx="0" iyy="0" izz="0" ixy="0" ixz="0" iyz="0"/>
-        </inertial>
-    </link>
-	<link name="T8_f2">
-        <inertial>
-            <mass value="0"/>
-            <origin xyz="0 0 0" rpy="0 0 0" />
-            <inertia ixx="0" iyy="0" izz="0" ixy="0" ixz="0" iyz="0"/>
-        </inertial>
-    </link>
-	<link name="T8">
-        <inertial>
-            <mass value="2.488"/>
-			<!--COM origin wrt jT9T8-->
-            <origin xyz="0           0    0.059874" rpy="0 0 0" />
-            <inertia ixx="0.0035473" iyy="0.0067278" izz="0.0043289" ixy="0" ixz="0" iyz="0"/>
-        </inertial>
-        <visual>
-			<!--box origin wrt jT9T8-->
-            <origin xyz="0           0    0.059874" rpy="0 0 0" />
-            <geometry>
-                <box size="0.13457    0.052626     0.11975"/>
-            </geometry>
-            <material name="color"/>
-        </visual>
-        <collision>
-			<!--box origin wrt jT9T8-->
-            <origin xyz="0           0    0.059874" rpy="0 0 0" />
-            <geometry>
-                <box size="0.13457    0.052626     0.11975"/>
-            </geometry>
-        </collision>
-    </link>
-	<link name="Neck_f1">
-        <inertial>
-            <mass value="0"/>
-            <origin xyz="0 0 0" rpy="0 0 0" />
-            <inertia ixx="0" iyy="0" izz="0" ixy="0" ixz="0" iyz="0"/>
-        </inertial>
-    </link>
-	<link name="Neck_f2">
-        <inertial>
-            <mass value="0"/>
-            <origin xyz="0 0 0" rpy="0 0 0" />
-            <inertia ixx="0" iyy="0" izz="0" ixy="0" ixz="0" iyz="0"/>
-        </inertial>
-    </link>
-	<link name="Neck">
-        <inertial>
-            <mass value="0.7464"/>
-			<!--COM origin wrt jT1C7-->
-            <origin xyz="0           0    0.044626" rpy="0 0 0" />
-            <inertia ixx="0.0006461" iyy="0.0006461" izz="0.00030124" ixy="0" ixz="0" iyz="0"/>
-        </inertial>
-        <visual>
-			<!--box origin wrt jT1C7-->
-            <origin xyz="0           0    0.044626" rpy="0 0 0" />
-            <geometry>
-		<cylinder length="0.089252" radius="0.014205"/>
-            </geometry>
-            <material name="color"/>
-        </visual>
-        <collision>
-			<!--box origin wrt jT1C7-->
-            <origin xyz="0           0    0.044626" rpy="0 0 0" />
-            <geometry>
-                <cylinder length="0.089252" radius="0.014205"/>
-            </geometry>
-        </collision>
-    </link>
-	<link name="Head_f1">
-        <inertial>
-            <mass value="0"/>
-            <origin xyz="0 0 0" rpy="0 0 0" />
-            <inertia ixx="0" iyy="0" izz="0" ixy="0" ixz="0" iyz="0"/>
-        </inertial>
-    </link>
-	<link name="Head_f2">
-        <inertial>
-            <mass value="0"/>
-            <origin xyz="0 0 0" rpy="0 0 0" />
-            <inertia ixx="0" iyy="0" izz="0" ixy="0" ixz="0" iyz="0"/>
-        </inertial>
-    </link>
-	<link name="Head">
-        <inertial>
-            <mass value="2.2392"/>
-			<!--COM origin wrt jC1Head-->
-            <origin xyz="0           0    0.089005" rpy="0 0 0" />
-            <inertia ixx="0.0070955" iyy="0.0070955" izz="0.0070955" ixy="0" ixz="0" iyz="0"/>
-        </inertial>
-        <visual>
-			<!--boc origin wrt jC1Head-->
-            <origin xyz="0           0    0.089005" rpy="0 0 0" />
-            <geometry>
-                <sphere radius="0.089005"/>
-            </geometry>
-            <material name="color"/>
-        </visual>
-        <collision>
-			<!--box origin wrt jC1Head-->
-            <origin xyz="0           0    0.089005" rpy="0 0 0" />
-            <geometry>
-                <sphere radius="0.089005"/>
-            </geometry>
-        </collision>
-    </link>
-	<!--Chain from (8) to (11)-->
-	<link name="RightShoulder_f1">
-        <inertial>
-            <mass value="0"/>
-            <origin xyz="0 0 0" rpy="0 0 0" />
-            <inertia ixx="0" iyy="0" izz="0" ixy="0" ixz="0" iyz="0"/>
-        </inertial>
-    </link>
-	<link name="RightShoulder_f2">
-        <inertial>
-            <mass value="0"/>
-            <origin xyz="0 0 0" rpy="0 0 0" />
-            <inertia ixx="0" iyy="0" izz="0" ixy="0" ixz="0" iyz="0"/>
-        </inertial>
-    </link>
-	<link name="RightShoulder">
-        <inertial>
-            <mass value="1.9282"/>
-			<!--COM origin wrt jRightC7Shoulder-->
-            <origin xyz="0   -0.065233           0" rpy="0 0 0" />
-            <inertia ixx="0.0030029" iyy="0.00053578" izz="0.0030029" ixy="0" ixz="0" iyz="0"/>
-        </inertial>
-        <visual>
-			<!--box origin wrt jRightC7Shoulder. RPY rotated of pi/2.-->
-            <origin xyz="0   -0.065233           0" rpy="1.5708 0 0" />
-            <geometry>
-                <cylinder length="0.13047" radius="0.023574"/>
-            </geometry>
-            <material name="color"/>
-        </visual>
-        <collision>
-			<!--box origin wrt jRightC7Shoulder. RPY rotated of pi/2.-->
-            <origin xyz="0   -0.065233           0" rpy="1.5708 0 0" />
-            <geometry>
-                <cylinder length="0.13047" radius="0.023574"/>
-            </geometry>
-        </collision>
-    </link>
-	<link name="RightUpperArm_f1">
-        <inertial>
-            <mass value="0"/>
-            <origin xyz="0 0 0" rpy="0 0 0" />
-            <inertia ixx="0" iyy="0" izz="0" ixy="0" ixz="0" iyz="0"/>
-        </inertial>
-    </link>
-	<link name="RightUpperArm_f2">
-        <inertial>
-            <mass value="0"/>
-            <origin xyz="0 0 0" rpy="0 0 0" />
-            <inertia ixx="0" iyy="0" izz="0" ixy="0" ixz="0" iyz="0"/>
-        </inertial>
-    </link>
-    <link name="RightUpperArm">
-        <inertial>
-            <mass value="1.866"/>
-			<!--COM origin wrt jRightShoulder-->
-            <origin xyz="0    -0.13497           0" rpy="0 0 0" />
-            <inertia ixx="0.011736" iyy="0.00080917" izz="0.011736" ixy="0" ixz="0" iyz="0"/>
-        </inertial>
-        <visual>
-			<!--box origin wrt jRightShoulder. RPY rotated of pi/2.-->
-            <origin xyz="0    -0.13497           0" rpy="1.5708 0 0" />
-            <geometry>
-                <cylinder length="0.26994" radius="0.029449"/>
-            </geometry>
-            <material name="color"/>
-        </visual>
-        <collision>
-			<!--box origin wrt jRightShoulder. RPY rotated of pi/2.-->
-            <origin xyz="0    -0.13497           0" rpy="1.5708 0 0" />
-            <geometry>
-                <cylinder length="0.26994" radius="0.029449"/>
-            </geometry>
-        </collision>
-    </link>
-	<link name="RightForeArm_f1">
-        <inertial>
-            <mass value="0"/>
-            <origin xyz="0 0 0" rpy="0 0 0" />
-            <inertia ixx="0" iyy="0" izz="0" ixy="0" ixz="0" iyz="0"/>
-        </inertial>
-    </link>
-	<link name="RightForeArm_f2">
-        <inertial>
-            <mass value="0"/>
-            <origin xyz="0 0 0" rpy="0 0 0" />
-            <inertia ixx="0" iyy="0" izz="0" ixy="0" ixz="0" iyz="0"/>
-        </inertial>
-    </link>
-	<link name="RightForeArm">
-        <inertial>
-            <mass value="1.244"/>
-			<!--COM origin wrt jRightElbow-->
-            <origin xyz="0    -0.11124           0" rpy="0 0 0" />
-            <inertia ixx="0.0052508" iyy="0.00023975" izz="0.0052508" ixy="0" ixz="0" iyz="0"/>
-        </inertial>
-        <visual>
-			<!--box origin wrt jRightElbow. RPY rotated of pi/2.-->
-            <origin xyz="0    -0.11124           0" rpy="1.5708 0 0" />
-            <geometry>
-                <cylinder length="0.22247" radius="0.019633"/>
-            </geometry>
-            <material name="color"/>
-        </visual>
-        <collision>
-			<!--box origin wrt jRightElbow. RPY rotated of pi/2.-->
-            <origin xyz="0    -0.11124           0" rpy="1.5708 0 0" />
-            <geometry>
-                <cylinder length="0.22247" radius="0.019633"/>
-            </geometry>
-        </collision>
-    </link>
-	<link name="RightHand_f1">
-        <inertial>
-            <mass value="0"/>
-            <origin xyz="0 0 0" rpy="0 0 0" />
-            <inertia ixx="0" iyy="0" izz="0" ixy="0" ixz="0" iyz="0"/>
-        </inertial>
-    </link>
-	<link name="RightHand_f2">
-        <inertial>
-            <mass value="0"/>
-            <origin xyz="0 0 0" rpy="0 0 0" />
-            <inertia ixx="0" iyy="0" izz="0" ixy="0" ixz="0" iyz="0"/>
-        </inertial>
-    </link>
-	<link name="RightHand">
-        <inertial>
-            <mass value="0.3732"/>
-			<!--COM origin wrt jRightWrist-->
-            <origin xyz="0   -0.083588           0" rpy="0 0 0" />
-            <inertia ixx="0.00091713" iyy="0.00043425" izz="0.0012555" ixy="0" ixz="0" iyz="0"/>
-        </inertial>
-        <visual>
-			<!--box origin wrt jRightWrist-->
-            <origin xyz="0   -0.083588           0" rpy="0 0 0" />
-            <geometry>
-                <box size="0.11145     0.16718    0.039266"/>
-            </geometry>
-            <material name="color"/>
-        </visual>
-        <collision>
-			<!--box origin wrt jRightWrist-->
-            <origin xyz="0   -0.083588           0" rpy="0 0 0" />
-            <geometry>
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
Commit message: Make human standing

File: wearable_robot_description/urdf/human_66dof.xacro (robot description, xacro)
@@ -690,5 +690,5 @@
       <origin xyz="0.054652           0   -0.039254" rpy="0 0 0" />
       <geometry>
-	<box size="0.17983    0.074775    0.078509"/>
+        <box size="0.17983    0.074775    0.078509"/>
       </geometry>
     </collision>
@@ -794,5 +794,5 @@
       <origin xyz="0           0    -0.20304" rpy="0 0 0" />
       <geometry>
-	<cylinder length="0.40608" radius="0.037388"/>
+        <cylinder length="0.40608" radius="0.037388"/>
       </geometry>
       <material name="color"/>
@@ -802,5 +802,5 @@
       <origin xyz="0           0    -0.20304" rpy="0 0 0" />
       <geometry>
-	<cylinder length="0.40608" radius="0.037388"/>
+        <cylinder length="0.40608" radius="0.037388"/>
       </geometry>
     </collision>
@@ -839,5 +839,5 @@
       <origin xyz="0.054652           0   -0.039254" rpy="0 0 0" />
       <geometry>
-	<box size="0.17983    0.074775    0.078509"/>
+        <box size="0.17983    0.074775    0.078509"/>
       </geometry>
     </collision>
@@ -882,5 +882,5 @@
   <!--JOINTS-->
   <!--Chain from (2) to (7)-->
-  <joint name="jL5S1_rotx" type="revolute">
+  <joint name="jL5S1_rotx" type="fixed">
     <origin xyz="-0.000206           0    0.098478" rpy="0 0 0"/>
     <parent link="Pelvis"/>
@@ -890,5 +890,5 @@
     <axis xyz="1 0 0" />
   </joint>
-  <joint name="jL5S1_roty" type="revolute">
+  <joint name="jL5S1_roty" type="fixed">
     <origin xyz="0 0 0" rpy="0 0 0"/>
     <parent link="L5_f1"/>
@@ -898,5 +898,5 @@
     <axis xyz="0 1 0" />
   </joint>
-  <joint name="jL5S1_rotz" type="revolute">
+  <joint name="jL5S1_rotz" type="fixed">
     <origin xyz="0 0 0" rpy="0 0 0"/>
     <parent link="L5_f2"/>
@@ -906,5 +906,5 @@
     <axis xyz="0 0 1" />
   </joint>
-  <joint name="jL4L3_rotx" type="revolute">
+  <joint name="jL4L3_rotx" type="fixed">
     <origin xyz="0.000374           0    0.095104" rpy="0 0 0"/>
     <parent link="L5"/>
@@ -914,5 +914,5 @@
     <axis xyz="1 0 0" />
   </joint>
-  <joint name="jL4L3_roty" type="revolute">
+  <joint name="jL4L3_roty" type="fixed">
     <origin xyz="0 0 0" rpy="0 0 0"/>
     <parent link="L3_f1"/>
@@ -922,5 +922,5 @@
     <axis xyz="0 1 0" />
   </joint>
-  <joint name="jL4L3_rotz" type="revolute">
+  <joint name="jL4L3_rotz" type="fixed">
     <origin xyz="0 0 0" rpy="0 0 0"/>
     <parent link="L3_f2"/>
@@ -930,5 +930,5 @@
     <axis xyz="0 0 1" />
   </joint>
-  <joint name="jL1T12_rotx" type="revolute">
+  <joint name="jL1T12_rotx" type="fixed">
     <origin xyz="0           0    0.085916" rpy="0 0 0"/>
     <parent link="L3"/>
@@ -938,5 +938,5 @@
     <axis xyz="1 0 0" />
   </joint>
-  <joint name="jL1T12_roty" type="revolute">
+  <joint name="jL1T12_roty" type="fixed">
     <origin xyz="0 0 0" rpy="0 0 0"/>
     <parent link="T12_f1"/>
@@ -946,5 +946,5 @@
     <axis xyz="0 1 0" />
   </joint>
-  <joint name="jL1T12_rotz" type="revolute">
+  <joint name="jL1T12_rotz" type="fixed">
     <origin xyz="0 0 0" rpy="0 0 0"/>
     <parent link="T12_f2"/>
@@ -954,5 +954,5 @@
     <axis xyz="0 0 1" />
   </joint>
-  <joint name="jT9T8_rotx" type="revolute">
+  <joint name="jT9T8_rotx" type="fixed">
     <origin xyz="0           0    0.085916" rpy="0 0 0"/>
     <parent link="T12"/>
@@ -962,5 +962,5 @@
     <axis xyz="1 0 0" />
   </joint>
-  <joint name="jT9T8_roty" type="revolute">
+  <joint name="jT9T8_roty" type="fixed">
     <origin xyz="0 0 0" rpy="0 0 0"/>
     <parent link="T8_f1"/>
@@ -970,5 +970,5 @@
     <axis xyz="0 1 0" />
   </joint>
-  <joint name="jT9T8_rotz" type="revolute">
+  <joint name="jT9T8_rotz" type="fixed">
     <origin xyz="0 0 0" rpy="0 0 0"/>
     <parent link="T8_f2"/>
@@ -978,5 +978,5 @@
     <axis xyz="0 0 1" />
   </joint>
-  <joint name="jT1C7_rotx" type="revolute">
+  <joint name="jT1C7_rotx" type="fixed">
     <origin xyz="0           0     0.11975" rpy="0 0 0"/>
     <parent link="T8"/>
@@ -986,5 +986,5 @@
     <axis xyz="1 0 0" />
   </joint>
-  <joint name="jT1C7_roty" type="revolute">
+  <joint name="jT1C7_roty" type="fixed">
     <origin xyz="0 0 0" rpy="0 0 0"/>
     <parent link="Neck_f1"/>
@@ -1002,5 +1002,5 @@
     <axis xyz="0 0 1" />
   </joint>
-  <joint name="jC1Head_rotx" type="revolute">
+  <joint name="jC1Head_rotx" type="fixed">
     <origin xyz="0.000152           0    0.089252" rpy="0 0 0"/>
     <parent link="Neck"/>
@@ -1010,5 +1010,5 @@
     <axis xyz="1 0 0" />
   </joint>
-  <joint name="jC1Head_roty" type="revolute">
+  <joint name="jC1Head_roty" type="fixed">
     <origin xyz="0 0 0" rpy="0 0 0"/>
     <parent link="Head_f1"/>
@@ -1027,5 +1027,6 @@
   </joint>
   <!--Chain from (8) to (11)-->
-  <joint name="jRightC7Shoulder_rotx" type="revolute">
+  <!-- Shouler -->
+  <joint name="jRightC7Shoulder_rotx" type="fixed">
     <origin xyz="0   -0.026313    0.067052" rpy="0 0 0"/>
     <parent link="T8"/>
@@ -1035,5 +1036,5 @@
     <axis xyz="1 0 0" />
   </joint>
-  <joint name="jRightC7Shoulder_roty" type="revolute">
+  <joint name="jRightC7Shoulder_roty" type="fixed">
     <origin xyz="0 0 0" rpy="0 0 0"/>
     <parent link="RightShoulder_f1"/>
@@ -1043,5 +1044,5 @@
     <axis xyz="0 1 0" />
   </joint>
-  <joint name="jRightC7Shoulder_rotz" type="revolute">
+  <joint name="jRightC7Shoulder_rotz" type="fixed">
     <origin xyz="0 0 0" rpy="0 0 0"/>
     <parent link="RightShoulder_f2"/>
@@ -1059,5 +1060,5 @@
     <axis xyz="1 0 0" />
   </joint>
-  <joint name="jRightShoulder_roty" type="revolute">
+  <joint name="jRightShoulder_roty" type="fixed">
     <origin xyz="0 0 0" rpy="0 0 0"/>
     <parent link="RightUpperArm_f1"/>
@@ -1083,5 +1084,5 @@
     <axis xyz="1 0 0" />
   </joint>
-  <joint name="jRightElbow_roty" type="revolute">
+  <joint name="jRightElbow_roty" type="fixed">
     <origin xyz="0 0 0" rpy="0 0 0"/>
     <parent link="RightForeArm_f1"/>
@@ -1130,5 +1131,5 @@
   </joint>
   <!--Chain from (12) to (15)-->
-  <joint name="jLeftC7Shoulder_rotx" type="revolute">
+  <joint name="jLeftC7Shoulder_rotx" type="fixed">
     <origin xyz="0    0.026313    0.067052" rpy="0 0 0"/>
     <parent link="T8"/>
@@ -1138,5 +1139,5 @@
     <axis xyz="1 0 0" />
   </joint>
-  <joint name="jLeftC7Shoulder_roty" type="revolute">
+  <joint name="jLeftC7Shoulder_roty" type="fixed">
     <origin xyz="0 0 0" rpy="0 0 0"/>
     <parent link="LeftShoulder_f1"/>
@@ -1146,5 +1147,5 @@
     <axis xyz="0 1 0" />
   </joint>
-  <joint name="jLeftC7Shoulder_rotz" type="revolute">
+  <joint name="jLeftC7Shoulder_rotz" type="fixed">
     <origin xyz="0 0 0" rpy="0 0 0"/>
     <parent link="LeftShoulder_f2"/>
