Commit message: Add arm link band points

File: wearable_robot_description/urdf/eduexo_v2.xacro (robot description, xacro)
@@ -73,5 +73,5 @@
       </inertial>
     </link>
-    <joint name="arm_band_link_fix_to_arm_link" type="fixed">
+    <joint name="arm_band_link_to_arm_link" type="fixed">
       <origin xyz="0.05 -0.05 0.2875" rpy="0 0 1.570796"/>
       <axis xyz="0 0 0" />
@@ -108,4 +108,85 @@
         <inertia ixx="1e-2" iyy="1e-2" izz="1e-2" ixy="0" ixz="0" iyz="0"/>
       </inertial>
+    </link>
+    <!-- band point -->
+    <joint name="arm_band_point_1_to_arm_link" type="fixed">
+      <origin xyz="0.05 -0.05 0.2875" rpy="0 0 1.570796"/>
+      <axis xyz="0 0 0" />
+      <parent link="arm_link"/>
+      <child link="arm_band_point_1"/>
+    </joint>
+    <joint name="arm_band_point_2_to_arm_link" type="fixed">
+      <origin xyz="0.05 -0.05 0.2875" rpy="0 0 1.570796"/>
+      <axis xyz="0 0 0" />
+      <parent link="arm_link"/>
+      <child link="arm_band_point_2"/>
+    </joint>
+    <joint name="arm_band_point_3_to_arm_link" type="fixed">
+      <origin xyz="0.05 -0.05 0.2875" rpy="0 0 1.570796"/>
+      <axis xyz="0 0 0" />
+      <parent link="arm_link"/>
+      <child link="arm_band_point_3"/>
+    </joint>
+    <joint name="arm_band_point_4_to_arm_link" type="fixed">
+      <origin xyz="0.05 -0.05 0.2875" rpy="0 0 1.570796"/>
+      <axis xyz="0 0 0" />
+      <parent link="arm_link"/>
+      <child link="arm_band_point_4"/>
+    </joint>
+    <link name="arm_band_point_1">
+      <visual>
+        <geometry>
+          <box size="0.004 0.004 0.004" />
+        </geometry>
+        <origin rpy="0 0 0" xyz="0.020 0.01 0.02"/>
+      </visual>
+      <collision>
+        <geometry>
+          <box size="0.004 0.004 0.004" />
+        </geometry>
+        <origin rpy="0 0 0" xyz="0.020 0.01 0.02"/>
+      </collision>
+    </link>
+    <link name="arm_band_point_2">
+      <visual>
+        <geometry>
+          <box size="0.004 0.004 0.004" />
+        </geometry>
+        <origin rpy="0 0 0" xyz="0.080 0.01 0.02"/>
+      </visual>
+      <collision>
+        <geometry>
+          <box size="0.004 0.004 0.004" />
+        </geometry>
+        <origin rpy="0 0 0" xyz="0.080 0.01 0.02"/>
+      </collision>
+    </link>
+    <link name="arm_band_point_3">
+      <visual>
+        <geometry>
+          <box size="0.004 0.004 0.004" />
+        </geometry>
+        <origin rpy="0 0 0" xyz="0.05 -0.020 0.02"/>
+      </visual>
+      <collision>
+        <geometry>
+          <box size="0.004 0.004 0.004" />
+        </geometry>
+        <origin rpy="0 0 0" xyz="0.05 -0.020 0.02"/>
+      </collision>
+    </link>
+    <link name="arm_band_point_4">
+      <visual>
+        <geometry>
+          <box size="0.004 0.004 0.004" />
+        </geometry>
+        <origin rpy="0 0 0" xyz="0.05 0.040 0.02"/>
+      </visual>
+      <collision>
+        <geometry>
+          <box size="0.004 0.004 0.004" />
+        </geometry>
+        <origin rpy="0 0 0" xyz="0.05 0.040 0.02"/>
+      </collision>
     </link>
   <ros2_control name="GazeboSystem" type="system">
@@ -118,5 +199,7 @@
         <param name="max">6.28</param>
       </command_interface>
-      <state_interface name="position"/>
+      <state_interface name="position">
+	<param name="initial_value">1.57079</param>
+      </state_interface>
       <state_interface name="velocity"/>
     </joint>
