Commit message: Add human 45 model and controller

File: wearable_robot_description/urdf/human_45dof.xacro (robot description, xacro)
@@ -1,4 +1,5 @@
 <?xml version="1.0"?>
 <robot  xmlns:xacro="http://www.ros.org/wiki/xacro"  name="dumpUrdf">
+  <xacro:include filename="$(find wearable_robot_description)/urdf/human_45dof.gazebo"/>
 <material name="orange">
   <color rgba="${255/255} ${108/255} ${10/255} 1.0"/>
@@ -85,4 +86,10 @@
 	</visual>
 </xacro:macro>
+  <!-- <link name="world"/> -->
+  <!-- <joint name="world_to_baselink_fixed" type="fixed"> -->
+  <!--   <parent link="world" /> -->
+  <!--   <child  link = "base_link" /> -->
+  <!--   <origin xyz="0 0 0" rpy="0 0 0" /> -->
+  <!-- </joint> -->
 	<link name="base_link">
 	</link>
@@ -345,3 +352,148 @@
 		<origin rpy = "0 0 0" xyz = "0.000000 -0.258947 0.000000" />
 	</joint>
+  <ros2_control name="GazeboSystem" type="system">
+    <hardware>
+      <plugin>gazebo_ros2_control/GazeboSystem</plugin>
+    </hardware>
+    <joint name="j_root_chest_joint1">
+      <command_interface name="position">
+      </command_interface>
+      <state_interface name="position"/>
+    </joint>
+    <joint name="j_root_chest_joint2">
+      <command_interface name="position">
+      </command_interface>
+      <state_interface name="position"/>
+    </joint>
+    <joint name="j_root_chest_joint3">
+      <command_interface name="position">
+      </command_interface>
+      <state_interface name="position"/>
+    </joint>
+    <joint name="j_chest_neck_joint1">
+      <command_interface name="position">
+      </command_interface>
+      <state_interface name="position"/>
+    </joint>
+    <joint name="j_chest_neck_joint2">
+      <command_interface name="position">
+      </command_interface>
+      <state_interface name="position"/>
+    </joint>
+    <joint name="j_chest_neck_joint3">
+      <command_interface name="position">
+      </command_interface>
+      <state_interface name="position"/>
+    </joint>
+    <joint name="j_root_right_hip_joint1">
+      <command_interface name="position">
+      </command_interface>
+      <state_interface name="position"/>
+    </joint>
+    <joint name="j_root_right_hip_joint2">
+      <command_interface name="position">
+      </command_interface>
+      <state_interface name="position"/>
+    </joint>
+    <joint name="j_root_right_hip_joint3">
+      <command_interface name="position">
+      </command_interface>
+      <state_interface name="position"/>
+    </joint>
+    <joint name="j_right_knee">
+      <command_interface name="position">
+      </command_interface>
+      <state_interface name="position"/>
+    </joint>
+    <joint name="j_right_knee_right_ankle_joint1">
+      <command_interface name="position">
+      </command_interface>
+      <state_interface name="position"/>
+    </joint>
+    <joint name="j_right_knee_right_ankle_joint2">
+      <command_interface name="position">
+      </command_interface>
+      <state_interface name="position"/>
+    </joint>
+    <joint name="j_right_knee_right_ankle_joint3">
+      <command_interface name="position">
+      </command_interface>
+      <state_interface name="position"/>
+    </joint>
+    <joint name="j_chest_right_shoulder_joint1">
+      <command_interface name="position">
+      </command_interface>
+      <state_interface name="position"/>
+    </joint>
+    <joint name="j_chest_right_shoulder_joint2">
+      <command_interface name="position">
+      </command_interface>
+      <state_interface name="position"/>
+    </joint>
+    <joint name="j_chest_right_shoulder_joint3">
+      <command_interface name="position">
+      </command_interface>
+      <state_interface name="position"/>
+    </joint>
+    <joint name="j_right_elbow">
+      <command_interface name="position">
+      </command_interface>
+      <state_interface name="position"/>
+    </joint>
+    <joint name="j_root_left_hip_joint1">
+      <command_interface name="position">
+      </command_interface>
+      <state_interface name="position"/>
+    </joint>
+    <joint name="j_root_left_hip_joint2">
+      <command_interface name="position">
+      </command_interface>
+      <state_interface name="position"/>
+    </joint>
+    <joint name="j_root_left_hip_joint3">
+      <command_interface name="position">
+      </command_interface>
+      <state_interface name="position"/>
+    </joint>
+    <joint name="j_left_knee">
+      <command_interface name="position">
+      </command_interface>
+      <state_interface name="position"/>
+    </joint>
+    <joint name="j_left_knee_left_ankle_joint1">
+      <command_interface name="position">
+      </command_interface>
+      <state_interface name="position"/>
+    </joint>
+    <joint name="j_left_knee_left_ankle_joint2">
+      <command_interface name="position">
+      </command_interface>
+      <state_interface name="position"/>
+    </joint>
+    <joint name="j_left_knee_left_ankle_joint3">
+      <command_interface name="position">
+      </command_interface>
+      <state_interface name="position"/>
+    </joint>
+    <joint name="j_chest_left_shoulder_joint1">
+      <command_interface name="position">
+      </command_interface>
+      <state_interface name="position"/>
+    </joint>
+    <joint name="j_chest_left_shoulder_joint2">
+      <command_interface name="position">
+      </command_interface>
+      <state_interface name="position"/>
+    </joint>
+    <joint name="j_chest_left_shoulder_joint3">
+      <command_interface name="position">
+      </command_interface>
+      <state_interface name="position"/>
+    </joint>
+    <joint name="j_left_elbow">
+      <command_interface name="position">
+      </command_interface>
+      <state_interface name="position"/>
+    </joint>
+  </ros2_control>
 </robot>

Commit message: Add human models from zento

File: wearable_robot_description/urdf/human_45dof.xacro (robot description, xacro)
@@ -2,7 +2,4 @@
 <robot  xmlns:xacro="http://www.ros.org/wiki/xacro"  name="dumpUrdf">
   <xacro:include filename="$(find wearable_robot_description)/urdf/human_45dof.gazebo"/>
-<material name="orange">
-  <color rgba="${255/255} ${108/255} ${10/255} 1.0"/>
-</material>
 <xacro:macro name="ball_joint" params="parent child limit effort_limit *origin">
   <link name="${parent}_${child}_link1">
@@ -86,270 +83,11 @@
 	</visual>
 </xacro:macro>
-  <!-- <link name="world"/> -->
-  <!-- <joint name="world_to_baselink_fixed" type="fixed"> -->
-  <!--   <parent link="world" /> -->
-  <!--   <child  link = "base_link" /> -->
-  <!--   <origin xyz="0 0 0" rpy="0 0 0" /> -->
-  <!-- </joint> -->
-	<link name="base_link">
-	</link>
-	<link name="base" >
-	</link>
-	<joint name="j_base_base_link_rotation" type="fixed">
-		<parent link = "base_link" />
-		<child link="base" />
-		<origin rpy = "${pi/2} 0 0" xyz = "0 0 0" />
-	</joint>
-	<link name="root" >
-		<inertial>
-			<origin rpy = "0 0 0" xyz = "0.0 0.07 0.0" />
-			<mass value = "6.000000" />
-      		<inertia ixx="0.019440000000000002" ixy="0" ixz="0" iyy="0.019440000000000002" iyz="0" izz="0.019440000000000002"/>
-		</inertial>
-		<xacro:sphere_v_c radius="0.18">
-			<origin rpy = "0 0 0" xyz = "0.000000 0.070000 0.000000" />
-		</xacro:sphere_v_c>
-	</link>
-	<joint name="j_root" type="fixed" >
-		<parent link = "base" />
-		<child link="root" />
-		<origin rpy = "0 0 0" xyz = "0 0.000000 0.000000" />
-	</joint>
-	<link name="chest" >
-		<inertial>
-			<origin rpy = "0 0 0" xyz = "0.000000 0.120000 0.000000" />
-			<mass value = "14.000000" />
-      		<inertia ixx="0.06776000000000001" ixy="0" ixz="0" iyy="0.06776000000000001" iyz="0" izz="0.06776000000000001"/>
-		</inertial>
-		<xacro:sphere_v_c radius="0.22">
-			<origin rpy = "0 0 0" xyz = "0.000000 0.120000 0.000000" />
-		</xacro:sphere_v_c>
-	</link>
-	<xacro:ball_joint parent="root" child="chest" limit="1.2" effort_limit="200">
-		<origin rpy = "0 0 0" xyz = "0.000000 0.236151 0.000000" />
-	</xacro:ball_joint>
-	<link name="neck" >
-		<inertial>
-			<origin rpy = "0 0 0" xyz = "0.0 0.175 0.0" />
-			<mass value = "2.000000" />
-      		<inertia ixx="0.008405" ixy="0" ixz="0" iyy="0.008405" iyz="0" izz="0.008405"/>
-		</inertial>
-		<xacro:sphere_v_c radius="0.205">
-			<origin rpy = "0 0 0" xyz = "0.0 0.175 0.0" />
-		</xacro:sphere_v_c>
-	</link>
-	<xacro:ball_joint parent="chest" child="neck" limit="1" effort_limit="50" >
-		<origin rpy = "0 0 0" xyz = "0.000000 0.223894 0.000000" />
-	</xacro:ball_joint>
-	<link name="right_hip" >
-		<inertial>
-			<origin rpy = "0 0 0" xyz = "0.000000 -0.210000 0.000000" />
-			<mass value = "4.500000" />
-			<inertia ixx="0.037153124999999995" ixy="0.0" ixz="0.0" iyy="0.037153124999999995" iyz="0.0" izz="0.00680625"/>
-		</inertial>
-		<xacro:cylinder_v_c radius="0.11" length="0.3">
-				<origin rpy = "${pi/2} 0 0" xyz = "0.000000 -0.210000 0.000000" />
-		</xacro:cylinder_v_c>
-	</link>
-	<xacro:ball_joint parent="root" child="right_hip" limit="1.5" effort_limit="200">
-		<origin rpy = "0 0 0" xyz = "0.000000 0.000000 0.084887" />
-	</xacro:ball_joint>
-	<link name="right_knee" >
-		<inertial>
-			<origin rpy = "0 0 0" xyz = "0.000000 -0.200000 0.000000" />
-			<mass value = "3.000000" />
-			<inertia ixx = "0.1" ixy = "0" ixz = "0" iyy = "0.1" iyz = "0" izz = "0.1" />
-		</inertial>
-		<xacro:cylinder_v_c length="0.31" radius="0.1">
-			<origin rpy = "${pi/2} 0 0" xyz = "0.000000 -0.200000 0.000000" />
-		</xacro:cylinder_v_c>
-	</link>
-	<joint name="j_right_knee" type="revolute" >
-		<parent link="right_hip" />
-		<child link="right_knee" />
-		<limit effort="150.0" lower="-3.14" upper="0." velocity="0.5"/>
-		<origin rpy = "0 0 0" xyz = "0.000000 -0.421546 0.000000" />
-		<axis xyz = "0.000000 0.000000 1.000000" />
-	</joint>
-	<link name="right_ankle" >
-		<inertial>
-			<origin rpy = "0 0 0" xyz = "0.045 -0.00225 0.000000" />
-			<mass value = "1.000000" />
-			<inertia ixx="0.0009270833333333333" ixy="0.0" ixz="0.0" iyy="0.0028628333333333327" iyz="0.0" izz="0.003285749999999999"/>
-		</inertial>
-		<xacro:box_v_c x="0.127" y="0.055" z = "0.09">
-			<origin rpy = "0 0 0" xyz = "0.045 -0.00225 0.000000"  />
-		</xacro:box_v_c>
-	</link>
-	<joint name="j_right_toe" type="fixed" >
-		<parent link="right_ankle" />
-		<child link="right_toe" />
-		<limit effort="150.0" lower="-3.14" upper="0." velocity="0.5"/>
-		<origin rpy = "0 0 0" xyz = "0.1 0.0 0.0" />
-		<axis xyz = "0.000000 0.000000 1.000000" />
-	</joint>
-	<link name="right_toe" >
-		<inertial>
-			<origin rpy = "0 0 0" xyz = "0.045 0.0 0.0" />
-			<mass value = "0.3" />
-			<inertia ixx="0.0009270833333333333" ixy="0.0" ixz="0.0" iyy="0.0028628333333333327" iyz="0.0" izz="0.003285749999999999"/>
-		</inertial>
-		<xacro:box_v_c x="0.05" y="0.055" z = "0.09">
-				<origin rpy = "0 0 0" xyz = "0.045 0.0 0.0" />
-		</xacro:box_v_c>
-	</link>
-	<xacro:ball_joint parent="right_knee" child="right_ankle" limit="1.2" effort_limit="90">
-		<origin rpy = "0 0 0" xyz = "0.000000 -0.409870 0.000000" />
-	</xacro:ball_joint>
-	<link name="right_shoulder" >
-		<inertial>
-			<origin rpy = "0 0 0" xyz = "0.000000 -0.140000 0.000000" />
-			<mass value = "1.500000" />
-			<inertia ixx="0.004809374999999999" ixy="0.0" ixz="0.0" iyy="0.004809374999999999" iyz="0.0" izz="0.0015187500000000001"/>
-		</inertial>
-		<xacro:cylinder_v_c length="0.18" radius="0.09">
-			<origin rpy = "${pi/2} 0 0" xyz = "0.000000 -0.140000 0.000000" />
-		</xacro:cylinder_v_c>
-	</link>
-	<xacro:ball_joint parent="chest" child="right_shoulder" limit="3.14" effort_limit="100">
-		<origin rpy = "0 0 0" xyz = "-0.02406 0.24350 0.18311" />
-	</xacro:ball_joint>
-	<link name="right_elbow" >
-		<inertial>
-			<origin rpy = "0 0 0" xyz = "0.000000 -0.120000 0.000000" />
-			<mass value = "1.000000" />
-			<inertia ixx="0.0019187499999999999" ixy="0.0" ixz="0.0" iyy="0.0019187499999999999" iyz="0.0" izz="0.0008"/>
-		</inertial>
-		<xacro:cylinder_v_c length="0.135" radius="0.08">
-				<origin rpy = "${pi/2} 0 0" xyz = "0.0 -0.12 0.0" />
-		</xacro:cylinder_v_c>
-	</link>
-	<joint name="j_right_elbow" type="revolute" >
-		<parent link="right_shoulder" />
-		<child link="right_elbow" />
-		<limit effort="60.0" lower="0" upper="3.14" velocity="0.5"/>
-		<origin rpy = "0 0 0" xyz = "0.000000 -0.274788 0.000000" />
-		<axis xyz = "0.000000 0.000000 1.000000" />
-	</joint>
-	<link name="right_wrist" >
-		<inertial>
-			<origin rpy = "0 0 0" xyz = "0.000000 0.000000 0.000000" />
-			<mass value = "0.500000" />
-			<inertia ixx="0.00032" ixy="0" ixz="0" iyy="0.00032" iyz="0" izz="0.00032"/>
-		</inertial>
-		<xacro:sphere_v_c radius="0.08">
-			<origin rpy = "0 0 0" xyz = "0.000000 0.000000 0.000000" />
-		</xacro:sphere_v_c>
-	</link>
-	<joint name="j_right_wrist" type="fixed" >
-		<parent link="right_elbow" />
-		<child link="right_wrist" />
-		<origin rpy = "0 0 0" xyz = "0.000000 -0.258947 0.000000" />
-	</joint>
-	<link name="left_hip" >
-		<inertial>
-			<origin rpy = "0 0 0" xyz = "0.000000 -0.210000 0.000000" />
-			<mass value = "4.500000" />
-			<inertia ixx="0.037153124999999995" ixy="0.0" ixz="0.0" iyy="0.037153124999999995" iyz="0.0" izz="0.00680625"/>
-		</inertial>
-		<xacro:cylinder_v_c length="0.3" radius="0.11">
-				<origin rpy = "${pi/2} 0 0" xyz = "0.000000 -0.210000 0.000000" />
-		</xacro:cylinder_v_c>
-	</link>
-	<xacro:ball_joint parent="root" child="left_hip" limit="1.5" effort_limit="200">
-		<origin rpy = "0 0 0" xyz = "0.000000 0.000000 -0.084887" />
-	</xacro:ball_joint>
-	<link name="left_knee" >
-		<inertial>
-			<origin rpy = "0 0 0" xyz = "0.000000 -0.200000 0.000000" />
-			<mass value = "3.000000" />
-			<inertia ixx="0.025900000000000003" ixy="0.0" ixz="0.0" iyy="0.025900000000000003" iyz="0.0" izz="0.0037500000000000007"/>
-		</inertial>
-		<xacro:cylinder_v_c length="0.31" radius="0.10000">
-				<origin rpy = "${pi/2} 0 0" xyz = "0.000000 -0.200000 0.000000" />
-		</xacro:cylinder_v_c>
-	</link>
-	<joint name="j_left_knee" type="revolute" >
-		<parent link="left_hip" />
-		<child link="left_knee" />
-		<limit effort="150.0" lower="-3.14" upper="0." velocity="0.5"/>
-		<origin rpy = "0 0 0" xyz = "0.000000 -0.421546 0.000000" />
-		<axis xyz = "0.000000 0.000000 1.000000" />
-	</joint>
-	<link name="left_ankle" >
-		<inertial>
-			<origin rpy = "0 0 0" xyz = "0.045 -0.00225 0.0" />
-			<mass value = "0.7" />
-			<inertia ixx="0.0009270833333333333" ixy="0.0" ixz="0.0" iyy="0.0028628333333333327" iyz="0.0" izz="0.003285749999999999"/>
-		</inertial>
-		<xacro:box_v_c x="0.127" y="0.055" z = "0.09">
-				<origin rpy = "0 0 0" xyz = "0.045 -0.00225 0.0" />
-		</xacro:box_v_c>
-	</link>
-	<joint name="j_left_toe" type="fixed" >
-		<parent link="left_ankle" />
-		<child link="left_toe" />
-		<limit effort="150.0" lower="-3.14" upper="0." velocity="0.5"/>
-		<origin rpy = "0 0 0" xyz = "0.1 0.0 0.0" />
-		<axis xyz = "0.000000 0.000000 1.000000" />
-	</joint>
-	<link name="left_toe" >
-		<inertial>
-			<origin rpy = "0 0 0" xyz = "0.045 0.0 0.0" />
-			<mass value = "0.3" />
-			<inertia ixx="0.0009270833333333333" ixy="0.0" ixz="0.0" iyy="0.0028628333333333327" iyz="0.0" izz="0.003285749999999999"/>
-		</inertial>
-		<xacro:box_v_c x="0.05" y="0.055" z = "0.09">
-				<origin rpy = "0 0 0" xyz = "0.045 0.0 0.0" />
-		</xacro:box_v_c>
-	</link>
-	<xacro:ball_joint parent="left_knee" child="left_ankle" limit="1.2" effort_limit="90">
-		<origin rpy = "0 0 0" xyz = "0.000000 -0.40987 0.000000" />
-	</xacro:ball_joint>
-	<link name="left_shoulder" >
-		<inertial>
-			<origin rpy = "0 0 0" xyz = "0.000000 -0.140000 0.000000" />
-			<mass value = "1.500000" />
-			<inertia ixx="0.004809374999999999" ixy="0.0" ixz="0.0" iyy="0.004809374999999999" iyz="0.0" izz="0.0015187500000000001"/>
-		</inertial>
-		<xacro:cylinder_v_c length="0.18" radius="0.09">
-			<origin rpy = "${pi/2} 0 0" xyz = "0.000000 -0.140000 0.000000" />
-		</xacro:cylinder_v_c>
-	</link>
-	<xacro:ball_joint parent="chest" child="left_shoulder" limit="3.14" effort_limit="100">
-		<origin rpy = "0 0 0" xyz = "-0.02405 0.24350 -0.18311" />
-	</xacro:ball_joint>
-	<link name="left_elbow" >
-		<inertial>
-			<origin rpy = "0 0 0" xyz = "0.000000 -0.12 0.000000" />
-			<mass value = "1.000000" />
-			<inertia ixx="0.0019187499999999999" ixy="0.0" ixz="0.0" iyy="0.0019187499999999999" iyz="0.0" izz="0.0008"/>
-		</inertial>
-		<xacro:cylinder_v_c length="0.135" radius="0.08">
-			<origin rpy = "${pi/2} 0 0" xyz = "0.000000 -0.12 0.000000" />
-		</xacro:cylinder_v_c>
-	</link>
-	<joint name="j_left_elbow" type="revolute" >
-		<parent link="left_shoulder" />
-		<child link="left_elbow" />
-		<limit effort="60.0" lower="0" upper="3.14" velocity="0.5"/>
-		<origin rpy = "0 0 0" xyz = "0.000000 -0.274788 0.000000" />
-		<axis xyz = "0.000000 0.000000 1.000000" />
-	</joint>
-	<link name="left_wrist" >
-		<inertial>
-			<origin rpy = "0 0 0" xyz = "0.000000 0.000000 0.000000" />
-			<mass value = "0.500000" />
-			<inertia ixx="0.00032" ixy="0" ixz="0" iyy="0.00032" iyz="0" izz="0.00032"/>
-		</inertial>
-		<xacro:sphere_v_c radius="0.08">
-			<origin rpy = "0 0 0" xyz = "0.000000 0.000000 0.000000" />
-		</xacro:sphere_v_c>
-	</link>
-	<joint name="j_left_wrist_joint" type="fixed" >
-		<parent link="left_elbow" />
-		<child link="left_wrist" />
-		<origin rpy = "0 0 0" xyz = "0.000000 -0.258947 0.000000" />
-	</joint>
+  <link name="world"/>
+  <joint name="world_to_baselink_fixed" type="fixed">
+    <parent link="world" />
+    <child  link = "base_link" />
+    <origin xyz="0 0 0" rpy="0 0 0" />
+  </joint>
+  <xacro:include filename="$(find wearable_robot_description)/urdf/humans/W0001.urdf"/>
   <ros2_control name="GazeboSystem" type="system">
     <hardware>

Commit message: Update human_45dof

File: wearable_robot_description/urdf/human_45dof.xacro (robot description, xacro)
@@ -229,9 +229,9 @@
       <state_interface name="position"/>
     </joint>
-    <joint name="j_left_elbow">
-      <command_interface name="position">
-      </command_interface>
-      <state_interface name="position"/>
-    </joint>
+    <!-- <joint name="j_left_elbow"> -->
+    <!--   <command_interface name="position"> -->
+    <!--   </command_interface> -->
+    <!--   <state_interface name="position"/> -->
+    <!-- </joint> -->
   </ros2_control>
 </robot>

File: wearable_robot_description/urdf/humans/W0001.urdf (robot description, URDF)
Before this commit: robot W0001, 35 links, 34 joints
Links:
- link left_elbow: geometry collision cylinder length=0.24 radius=0.04; visual cylinder length=0.25 radius=0.04
Joints:
- joint j_root_chest_joint1: limit lower=-1.2 upper=1.2 effort=200 velocity=3 -> (none); type revolute -> fixed
- joint j_root_chest_joint2: limit lower=-1.2 upper=1.2 effort=200 velocity=3 -> (none); type revolute -> fixed
- joint j_root_chest_joint3: limit lower=-1.2 upper=1.2 effort=200 velocity=3 -> (none); type revolute -> fixed
