Commit message: 휴먼 45dof 왼쪽암 joint 토크 제어
1. human_45dof.launch.py 실행
2. human_Arm_gazebo_effort_test 실행

File: wearable_robot_description/urdf/human_45dof.xacro (robot description, xacro)
@@ -94,144 +94,177 @@
       <plugin>gazebo_ros2_control/GazeboSystem</plugin>
     </hardware>
-    <joint name="j_root_chest_joint1">
-      <command_interface name="position">
+    <!-- <joint name="j_root_chest_joint1"> -->
+    <!--   <command_interface name="position"> -->
+    <!--   </command_interface> -->
+    <!--   <state_interface name="position"/> -->
+    <!-- </joint> -->
+    <!--  -->
+    <!-- <joint name="j_root_chest_joint2"> -->
+    <!--   <command_interface name="position"> -->
+    <!--   </command_interface> -->
+    <!--   <state_interface name="position"/> -->
+    <!-- </joint> -->
+    <!--  -->
+    <!-- <joint name="j_root_chest_joint3"> -->
+    <!--   <command_interface name="position"> -->
+    <!--   </command_interface> -->
+    <!--   <state_interface name="position"/> -->
+    <!-- </joint> -->
+    <!--  -->
+    <!-- <joint name="j_chest_neck_joint1"> -->
+    <!--   <command_interface name="position"> -->
+    <!--   </command_interface> -->
+    <!--   <state_interface name="position"/> -->
+    <!-- </joint> -->
+    <!--  -->
+    <!-- <joint name="j_chest_neck_joint2"> -->
+    <!--   <command_interface name="position"> -->
+    <!--   </command_interface> -->
+    <!--   <state_interface name="position"/> -->
+    <!-- </joint> -->
+    <!--  -->
+    <!-- <joint name="j_chest_neck_joint3"> -->
+    <!--   <command_interface name="position"> -->
+    <!--   </command_interface> -->
+    <!--   <state_interface name="position"/> -->
+    <!-- </joint> -->
+    <!--  -->
+    <!-- <joint name="j_root_right_hip_joint1"> -->
+    <!--   <command_interface name="position"> -->
+    <!--   </command_interface> -->
+    <!--   <state_interface name="position"/> -->
+    <!-- </joint> -->
+    <!--  -->
+    <!-- <joint name="j_root_right_hip_joint2"> -->
+    <!--   <command_interface name="position"> -->
+    <!--   </command_interface> -->
+    <!--   <state_interface name="position"/> -->
+    <!-- </joint> -->
+    <!--  -->
+    <!-- <joint name="j_root_right_hip_joint3"> -->
+    <!--   <command_interface name="position"> -->
+    <!--   </command_interface> -->
+    <!--   <state_interface name="position"/> -->
+    <!-- </joint> -->
+    <!--  -->
+    <!-- <joint name="j_right_knee"> -->
+    <!--   <command_interface name="position"> -->
+    <!--   </command_interface> -->
+    <!--   <state_interface name="position"/> -->
+    <!-- </joint> -->
+    <!--  -->
+    <!-- <joint name="j_right_knee_right_ankle_joint1"> -->
+    <!--   <command_interface name="position"> -->
+    <!--   </command_interface> -->
+    <!--   <state_interface name="position"/> -->
+    <!-- </joint> -->
+    <!--  -->
+    <!-- <joint name="j_right_knee_right_ankle_joint2"> -->
+    <!--   <command_interface name="position"> -->
+    <!--   </command_interface> -->
+    <!--   <state_interface name="position"/> -->
+    <!-- </joint> -->
+    <!--  -->
+    <!-- <joint name="j_right_knee_right_ankle_joint3"> -->
+    <!--   <command_interface name="position"> -->
+    <!--   </command_interface> -->
+    <!--   <state_interface name="position"/> -->
+    <!-- </joint> -->
+    <!--  -->
+    <!-- <joint name="j_chest_right_shoulder_joint1"> -->
+    <!--   <command_interface name="position"> -->
+    <!--   </command_interface> -->
+    <!--   <state_interface name="position"/> -->
+    <!-- </joint> -->
+    <!--  -->
+    <!-- <joint name="j_chest_right_shoulder_joint2"> -->
+    <!--   <command_interface name="position"> -->
+    <!--   </command_interface> -->
+    <!--   <state_interface name="position"/> -->
+    <!-- </joint> -->
+    <!--  -->
+    <!-- <joint name="j_chest_right_shoulder_joint3"> -->
+    <!--   <command_interface name="position"> -->
+    <!--   </command_interface> -->
+    <!--   <state_interface name="position"/> -->
+    <!-- </joint> -->
+    <!--  -->
+    <!-- <joint name="j_right_elbow"> -->
+    <!--   <command_interface name="position"> -->
+    <!--   </command_interface> -->
+    <!--   <state_interface name="position"/> -->
+    <!-- </joint> -->
+    <!--  -->
+    <!-- <joint name="j_root_left_hip_joint1"> -->
+    <!--   <command_interface name="position"> -->
+    <!--   </command_interface> -->
+    <!--   <state_interface name="position"/> -->
+    <!-- </joint> -->
+    <!--  -->
+    <!-- <joint name="j_root_left_hip_joint2"> -->
+    <!--   <command_interface name="position"> -->
+    <!--   </command_interface> -->
+    <!--   <state_interface name="position"/> -->
+    <!-- </joint> -->
+    <!--  -->
+    <!-- <joint name="j_root_left_hip_joint3"> -->
+    <!--   <command_interface name="position"> -->
+    <!--   </command_interface> -->
+    <!--   <state_interface name="position"/> -->
+    <!-- </joint> -->
+    <!--  -->
+    <!-- <joint name="j_left_knee"> -->
+    <!--   <command_interface name="position"> -->
+    <!--   </command_interface> -->
+    <!--   <state_interface name="position"/> -->
+    <!-- </joint> -->
+    <!--  -->
+    <!-- <joint name="j_left_knee_left_ankle_joint1"> -->
+    <!--   <command_interface name="position"> -->
+    <!--   </command_interface> -->
+    <!--   <state_interface name="position"/> -->
+    <!-- </joint> -->
+    <!--  -->
+    <!-- <joint name="j_left_knee_left_ankle_joint2"> -->
+    <!--   <command_interface name="position"> -->
+    <!--   </command_interface> -->
+    <!--   <state_interface name="position"/> -->
+    <!-- </joint> -->
+    <!--  -->
+    <!-- <joint name="j_left_knee_left_ankle_joint3"> -->
+    <!--   <command_interface name="position"> -->
+    <!--   </command_interface> -->
+    <!--   <state_interface name="position"/> -->
+    <!-- </joint> -->
+    <!--  -->
+    <!-- <joint name="j_chest_left_shoulder_joint1"> -->
+    <!--   <command_interface name="position"> -->
+    <!--   </command_interface> -->
+    <!--   <state_interface name="position"/> -->
+    <!-- </joint> -->
+    <!--  -->
+    <!-- <joint name="j_chest_left_shoulder_joint2"> -->
+    <!--   <command_interface name="position"> -->
+    <!--   </command_interface> -->
+    <!--   <state_interface name="position"/> -->
+    <!-- </joint> -->
+    <!--  -->
+    <!-- <joint name="j_chest_left_shoulder_joint3"> -->
+    <!--   <command_interface name="position"> -->
+    <!--   </command_interface> -->
+    <!--   <state_interface name="position"/> -->
+    <!-- </joint> -->
+    <joint name="j_left_elbow">
+      <command_interface name="effort">
+        <param name="min">-300.0</param>
+        <param name="max">+300.0</param>
       </command_interface>
+      <!-- <state_interface name="position"> -->
+			<!--   <param name="initial_value">1.57079</param>           -->
+      <!-- </state_interface> -->
       <state_interface name="position"/>
+      <state_interface name="velocity"/>
+      <state_interface name="effort"/>
     </joint>
-    <joint name="j_root_chest_joint2">
-      <command_interface name="position">
-      </command_interface>
-      <state_interface name="position"/>
-    </joint>
-    <joint name="j_root_chest_joint3">
-      <command_interface name="position">
-      </command_interface>
-      <state_interface name="position"/>
-    </joint>
-    <joint name="j_chest_neck_joint1">
-      <command_interface name="position">
-      </command_interface>
-      <state_interface name="position"/>
-    </joint>
-    <joint name="j_chest_neck_joint2">
-      <command_interface name="position">
-      </command_interface>
-      <state_interface name="position"/>
-    </joint>
-    <joint name="j_chest_neck_joint3">
-      <command_interface name="position">
-      </command_interface>
-      <state_interface name="position"/>
-    </joint>
-    <joint name="j_root_right_hip_joint1">
-      <command_interface name="position">
-      </command_interface>
-      <state_interface name="position"/>
-    </joint>
-    <joint name="j_root_right_hip_joint2">
-      <command_interface name="position">
-      </command_interface>
-      <state_interface name="position"/>
-    </joint>
-    <joint name="j_root_right_hip_joint3">
-      <command_interface name="position">
-      </command_interface>
-      <state_interface name="position"/>
-    </joint>
-    <joint name="j_right_knee">
-      <command_interface name="position">
-      </command_interface>
-      <state_interface name="position"/>
-    </joint>
-    <joint name="j_right_knee_right_ankle_joint1">
-      <command_interface name="position">
-      </command_interface>
-      <state_interface name="position"/>
-    </joint>
-    <joint name="j_right_knee_right_ankle_joint2">
-      <command_interface name="position">
-      </command_interface>
-      <state_interface name="position"/>
-    </joint>
-    <joint name="j_right_knee_right_ankle_joint3">
-      <command_interface name="position">
-      </command_interface>
-      <state_interface name="position"/>
-    </joint>
-    <joint name="j_chest_right_shoulder_joint1">
-      <command_interface name="position">
-      </command_interface>
-      <state_interface name="position"/>
-    </joint>
-    <joint name="j_chest_right_shoulder_joint2">
-      <command_interface name="position">
-      </command_interface>
-      <state_interface name="position"/>
-    </joint>
-    <joint name="j_chest_right_shoulder_joint3">
-      <command_interface name="position">
-      </command_interface>
-      <state_interface name="position"/>
-    </joint>
-    <joint name="j_right_elbow">
-      <command_interface name="position">
-      </command_interface>
-      <state_interface name="position"/>
-    </joint>
-    <joint name="j_root_left_hip_joint1">
-      <command_interface name="position">
-      </command_interface>
-      <state_interface name="position"/>
-    </joint>
-    <joint name="j_root_left_hip_joint2">
-      <command_interface name="position">
-      </command_interface>
-      <state_interface name="position"/>
-    </joint>
-    <joint name="j_root_left_hip_joint3">
-      <command_interface name="position">
-      </command_interface>
-      <state_interface name="position"/>
-    </joint>
-    <joint name="j_left_knee">
-      <command_interface name="position">
-      </command_interface>
-      <state_interface name="position"/>
-    </joint>
-    <joint name="j_left_knee_left_ankle_joint1">
-      <command_interface name="position">
-      </command_interface>
-      <state_interface name="position"/>
-    </joint>
-    <joint name="j_left_knee_left_ankle_joint2">
-      <command_interface name="position">
-      </command_interface>
-      <state_interface name="position"/>
-    </joint>
-    <joint name="j_left_knee_left_ankle_joint3">
-      <command_interface name="position">
-      </command_interface>
-      <state_interface name="position"/>
-    </joint>
-    <joint name="j_chest_left_shoulder_joint1">
-      <command_interface name="position">
-      </command_interface>
-      <state_interface name="position"/>
-    </joint>
-    <joint name="j_chest_left_shoulder_joint2">
-      <command_interface name="position">
-      </command_interface>
-      <state_interface name="position"/>
-    </joint>
-    <joint name="j_chest_left_shoulder_joint3">
-      <command_interface name="position">
-      </command_interface>
-      <state_interface name="position"/>
-    </joint>
-    <!-- <joint name="j_left_elbow"> -->
-    <!--   <command_interface name="position"> -->
-    <!--   </command_interface> -->
-    <!--   <state_interface name="position"/> -->
-    <!-- </joint> -->
   </ros2_control>
 </robot>
