Commit message: Update size of upper-limb's forearm band

File: wearable_robot_description/urdf/upper_limb.xacro (robot description, xacro)
@@ -67,5 +67,5 @@
       <collision>
         <geometry>
-          <mesh filename="$(find wearable_robot_description)/meshes/pipe.dae" scale="0.060 0.050 0.01"/>
+          <mesh filename="$(find wearable_robot_description)/meshes/pipe.dae" scale="0.060 0.055 0.01"/>
         </geometry>
         <!-- <origin rpy="1.570796 1.570796 0" xyz="0.0 -0.025 0.0"/> -->
