Commit message: 45dof 휴먼 모델 왼쪽 어깨 움직임 가용범위 조정 +- 0.01 radian

File: wearable_robot_description/urdf/humans/W0001.urdf (robot description, URDF)
Before this commit: robot W0001, 35 links, 34 joints
Joints:
- joint j_chest_left_shoulder_joint2: limit lower=-3.14 upper=3.14 effort=100 velocity=3 -> lower=-0.01 upper=0.01 effort=100 velocity=3
- joint j_chest_left_shoulder_joint3: limit lower=-3.14 upper=3.14 effort=100 velocity=3 -> lower=-0.01 upper=0.01 effort=100 velocity=3

Commit message: 45dof 휴먼 모델: 목 고정, joint 가용범위 줄임

File: wearable_robot_description/urdf/humans/W0001.urdf (robot description, URDF)
Before this commit: robot W0001, 35 links, 34 joints
Joints:
- joint j_chest_neck_joint1: limit lower=-1 upper=1 effort=50 velocity=3 -> lower=-0.01 upper=0.01 effort=50 velocity=3
- joint j_chest_neck_joint3: limit lower=-1 upper=1 effort=50 velocity=3 -> lower=-0.01 upper=0.01 effort=50 velocity=3

Commit message: 휴먼모델 왼쪽 암과 웨어러블(upper-limb) 디바이스 연결해서 토크제어  - 휴먼 모델 조인트 최대 토크, 속도, 마찰값 수정  - 디바이스 모델 조인트 최대 토크, 속도, 마찰값 수정  - 디바이스 착용에 맞춰서 PID 계수 수정  - 휴먼모델에서 디바이스 토크 읽어서 제어하도록 수정  - 김우진 박사님과 같이 작업하여 코드 수정

File: wearable_robot_description/urdf/humans/W0001.urdf (robot description, URDF)
Before this commit: robot W0001, 35 links, 34 joints
Links:
- link left_shoulder: geometry collision cylinder length=0.135 radius=0.045; visual cylinder length=0.26 radius=0.045
Joints:
- joint j_left_elbow: limit lower=0 upper=3.14 effort=60.0 velocity=0.5 -> lower=0 upper=3.14 effort=300.0 velocity=100

File: wearable_robot_description/urdf/upper_limb.xacro (robot description, xacro)
@@ -16,5 +16,5 @@
         </geometry>
         <!-- <origin rpy="0 0 -1.570796" xyz="0.0 0 0.0"/>  -->
-        <origin rpy="-3.141592 -1.570706 0" xyz="0.1 -0.05 0.00"/>
+        <origin rpy="-3.141592 -1.570796 0" xyz="0.1 -0.05 0.00"/>
         <material name="blue">
           <color rgba="0 0 1 1"/>
@@ -31,6 +31,6 @@
         <origin xyz="0 0 0.1575"/>
         <axis xyz="0 0 0" />
-        <limit effort="300" velocity="0.1" lower="-4.1" upper="-1.5"/>
-        <dynamics damping="50" friction="1"/>
+        <limit effort="500" velocity="100" lower="-4.1" upper="-1.570796"/>
+        <dynamics damping="1" friction="1"/>
     </joint>
     <link name="forearm_link">
@@ -60,16 +60,15 @@
         <geometry>
           <!-- <mesh filename="$(find wearable_robot_description)/meshes/pipe.dae" scale="0.03 0.03 0.01"/> -->
-          <mesh filename="$(find wearable_robot_description)/meshes/pipe.dae" scale="0.052 0.052 0.01"/>
-        </geometry>
-        <!-- <origin rpy="1.570796 1.570796 0" xyz="0.05 -0.025 0.0"/> -->
-        <origin rpy="1.570796 1.570796 0" xyz="-0.0250 -0.025 0.0"/>
+          <mesh filename="$(find wearable_robot_description)/meshes/pipe.dae" scale="0.050 0.050 0.01"/>
+        </geometry>
+        <!-- <origin rpy="1.570796 1.570796 0" xyz="0.0 -0.025 0.0"/> -->
+        <origin rpy="1.570796 1.570796 0" xyz="-0.0050 -0.025 0.0"/>
       </visual>
       <collision>
         <geometry>
-          <!-- <mesh filename="$(find wearable_robot_description)/meshes/pipe.dae" scale="0.03 0.03 0.01"/> -->
-          <mesh filename="$(find wearable_robot_description)/meshes/pipe.dae" scale="0.052 0.052 0.01"/>
-        </geometry>
-        <!-- <origin rpy="1.570796 1.570796 0" xyz="0.05 -0.025 0.0"/> -->
-        <origin rpy="1.570796 1.570796 0" xyz="-0.0250 -0.025 0.0"/>
+          <mesh filename="$(find wearable_robot_description)/meshes/pipe.dae" scale="0.060 0.050 0.01"/>
+        </geometry>
+        <!-- <origin rpy="1.570796 1.570796 0" xyz="0.0 -0.025 0.0"/> -->
+        <origin rpy="1.570796 1.570796 0" xyz="-0.0050 -0.025 0.0"/>
       </collision>
       <inertial>
@@ -87,30 +86,27 @@
       <visual>
         <geometry>
-          <!-- <mesh filename="$(find wearable_robot_description)/meshes/pipe.dae" scale="0.0295 0.0295 0.01"/> -->
-          <mesh filename="$(find wearable_robot_description)/meshes/pipe.dae" scale="0.05 0.05 0.01"/>
-        </geometry>
-        <origin rpy="0 0 0" xyz="0.05 0.01 0.02"/>
-      </visual>
-      <!-- <collision> -->
-      <!--   <geometry> -->
-      <!--     [> <mesh filename="$(find wearable_robot_description)/meshes/pipe.dae" scale="0.0295 0.0295 0.01"/> <] -->
-      <!--     <mesh filename="$(find wearable_robot_description)/meshes/pipe.dae" scale="0.07 0.07 0.01"/> -->
-      <!--   </geometry> -->
-      <!--   <origin rpy="0 0 0" xyz="0.05 0.01 0.02"/> -->
-      <!-- </collision> -->
-      <visual>
-        <geometry>
-          <!-- <mesh filename="$(find wearable_robot_description)/meshes/pipe.dae" scale="0.0295 0.0295 0.01"/> -->
-          <mesh filename="$(find wearable_robot_description)/meshes/pipe.dae" scale="0.05 0.05 0.01"/>
-        </geometry>
-        <origin rpy="0 0 0" xyz="0.05 0.01 -0.07"/>
-      </visual>
-      <!-- <collision> -->
-      <!--   <geometry> -->
-      <!--     [> <mesh filename="$(find wearable_robot_description)/meshes/pipe.dae" scale="0.0295 0.0295 0.01"/> <] -->
-      <!--     <mesh filename="$(find wearable_robot_description)/meshes/pipe.dae" scale="0.07 0.07 0.01"/> -->
-      <!--   </geometry> -->
-      <!--   <origin rpy="0 0 0" xyz="0.05 0.01 -0.07"/> -->
-      <!-- </collision> -->
+          <mesh filename="$(find wearable_robot_description)/meshes/pipe.dae" scale="0.05 0.05 0.02"/>
+        </geometry>
+          <!-- <origin rpy="0 0 0" xyz="0.05 0.01 0.02"/> --> <!-- x up dir, y left dir, z is z dir -->
+        <origin rpy="0 0 0" xyz="0.06 0.049 0.005"/>
+      </visual>
+      <collision>
+        <geometry>
+          <mesh filename="$(find wearable_robot_description)/meshes/pipe.dae" scale="0.045 0.045 0.02"/>
+        </geometry>
+        <origin rpy="0 0 0" xyz="0.06 0.049 0.005"/>
+      </collision>
+      <visual>
+        <geometry>
+          <mesh filename="$(find wearable_robot_description)/meshes/pipe.dae" scale="0.05 0.05 0.02"/>
+        </geometry>
+        <origin rpy="0 0 0" xyz="0.06 0.049 -0.05"/>
+      </visual>
+      <collision>
+        <geometry>
+          <mesh filename="$(find wearable_robot_description)/meshes/pipe.dae" scale="0.045 0.045 0.02"/>
+        </geometry>
+        <origin rpy="0 0 0" xyz="0.06 0.049 -0.05"/>
+      </collision>
       <inertial>
         <mass value="0.001"/>
@@ -214,5 +210,5 @@
       </command_interface>
       <state_interface name="position">
-	      <param name="initial_value">1.57079</param>
+	      <param name="initial_value">1.570796</param>
       </state_interface>
       <state_interface name="velocity"/>
